File: Radiator valve/BMS.kicad_sch (KiCad schematic)
At the start: 13 parts, among them J3 Conn_01x02, U5 BQ24075RGT

Commit message: Finished schematic
Parts:
- R18, R19: footprint Resistor_SMD:R_0603_1608Metric -> Resistor_SMD:R_0402_1005Metric
- TH1: now not fitted
Connections:
- net +BATT: now also U5.11 (OUT)
- net at BT1.1 (+), C5.1, U5.2 (BAT): now also U5.3 (BAT)
- net at D1.1 (K), U5.7 (~{PGOOD}): no longer U5.3 (BAT)
- no-connect marks 1 -> 3
Other:
- note removed: "BMS"
- note removed: "Tym sie nie zajmować raczej do wyjebania"
- moved on the sheet: BT1, C14, C18, C5, D1, D3, J3, R18, R19, R20, R21, U5
