File: Radiator valve/Radiator valve.kicad_pcb (KiCad board)
At the start: 2 copper layers, 40 x 40 mm, 39 parts, among them IC1 SC4626ZSKTRT, J1 53047-0410, J2 USB_C_Receptacle_USB2.0_14P, U1 MLX90632SLD-BCB-000-SP, U2 ESP32-S3-MINI-1, U5 BQ24075RGT, U6 DRV8833PW

Commit message: Finished schematic
Parts:
- removed C1: 10u, Capacitor_SMD:C_0603_1608Metric
- removed C13: 10u, Capacitor_SMD:C_0805_2012Metric
- removed FB1: 1u, Inductor_SMD:L_0603_1608Metric
- removed IC1: SC4626ZSKTRT, SC4626ZSKTRT:SOT95P280X145-5N
- removed L1: 2.2u, Inductor_SMD:L_0805_2012Metric
- removed R15: 5k1, Resistor_SMD:R_0603_1608Metric
- removed R18: 1.18k, Resistor_SMD:R_0603_1608Metric
- removed R19: 1.13k, Resistor_SMD:R_0603_1608Metric
- removed R20, R21: 1.5k, Resistor_SMD:R_0603_1608Metric
- removed U5: BQ24075RGT, Package_DFN_QFN:VQFN-16-1EP_3x3mm_P0.5mm_EP1.6x1.6mm
- added C10: 100n, Capacitor_SMD:C_0402_1005Metric, F.Cu at (72.3, 86.7)
- added C17: 10u, Capacitor_SMD:C_0402_1005Metric, F.Cu at (72.3, 88.7)
- added C19: 10u, Capacitor_SMD:C_0402_1005Metric, F.Cu at (72.3, 90.7)
- added C2: 10u, Capacitor_SMD:C_0603_1608Metric, F.Cu at (60.8, 70.2)
- added D2: LED_Small, LED_SMD:LED_0603_1608Metric, F.Cu at (81.0, 91.0)
- added D4: PESD5V0S1UL,315, Diode_SMD:D_SOD-523, F.Cu at (80.8, 85.5)
- added L2: 1.5u, Inductor_SMD:L_Coilcraft_LPS3010, F.Cu at (67.0, 88.1)
- added R1: 10k, Resistor_SMD:R_0402_1005Metric, F.Cu at (60.3, 82.5)
- added R10: 1.13k, Resistor_SMD:R_0402_1005Metric, F.Cu at (63.2, 86.4)
- added R11: 1.5k, Resistor_SMD:R_0603_1608Metric, F.Cu at (68.8, 75.2)
- added R12: 1.5k, Resistor_SMD:R_0603_1608Metric, F.Cu at (68.8, 77.7)
- added R9: 1.18k, Resistor_SMD:R_0402_1005Metric, F.Cu at (63.2, 84.5)
- added U3: TPS63031DSK, Package_SON:WSON-10-1EP_2.5x2.5mm_P0.5mm_EP1.2x2mm, F.Cu at (67.5, 83.8)
- added U4: BQ24075RGT, Package_DFN_QFN:VQFN-16-1EP_3x3mm_P0.5mm_EP1.6x1.6mm, F.Cu at (76.4, 84.5)
- C18: value 1u -> 4.7u
- C5: value 4.7u -> 1u
- C7, C8: footprint Capacitor_SMD:C_0603_1608Metric -> Capacitor_SMD:C_0402_1005Metric
- D3: value LED_Small -> PESD5V0S1UL,315; footprint LED_SMD:LED_0603_1608Metric -> Diode_SMD:D_SOD-523
- J2: footprint Connector_USB:USB_C_Receptacle_GCT_USB4125-xx-x-0190_6P_TopMnt_Horizontal -> Connector_USB:USB_C_Receptacle_GCT_USB4110
- R13, R14, R2, R3, R4, R7, R8: footprint Resistor_SMD:R_0603_1608Metric -> Resistor_SMD:R_0402_1005Metric
- R5: value 10k -> 5k1; footprint Resistor_SMD:R_0603_1608Metric -> Resistor_SMD:R_0402_1005Metric
- moved J2 77.4 mm to (130.3, 96.4), turned to 0 degrees
- moved U2 60.7 mm to (130.6, 69.8)
- moved C11 38.6 mm to (64.8, 70.2)
- moved C5 28.7 mm to (60.8, 75.2)
- moved C8 25.2 mm to (72.3, 84.8)
- moved D1 25.1 mm to (81.0, 88.4)
- moved C7 24.9 mm to (72.3, 82.8)
- moved C14 23.9 mm to (64.8, 75.2)
- moved C9 23.6 mm to (60.8, 80.2)
- moved C4 21.3 mm to (60.8, 72.7)
- moved R6 21.3 mm to (68.8, 72.7)
- moved J1 19.3 mm to (77.6, 71.6)
- moved C12 19.1 mm to (64.8, 72.7)
- moved C6 19.1 mm to (60.8, 77.7)
- moved R4 18.3 mm to (60.3, 88.4)
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Connections:
- C15 pad 1: Net-(C15-Pad1) -> VBUS
- C18 pad 1: GND -> Net-(C18-Pad1)
- C18 pad 2: VBUS -> GND
- C5 pad 1: Net-(C5-Pad1) -> GND
- C5 pad 2: GND -> VBUS
- D3 pad 1: Net-(D3-K) -> /USB_D-
- D3 pad 2: Net-(D3-A) -> unconnected-(D3-A-Pad2)
- J2 pad A9: Net-(C15-Pad1) -> VBUS
- J2 pad B9: Net-(C15-Pad1) -> VBUS
- R3 pad 1: /AIN2 -> /BIN1
- R3 pad 2: Net-(U6-AIN2) -> Net-(U6-BIN1)
- R4 pad 1: /BIN1 -> /BIN2
- R4 pad 2: Net-(U6-BIN1) -> Net-(U6-BIN2)
- R5 pad 1: /BIN2 -> Net-(J2-CC2)
- R5 pad 2: Net-(U6-BIN2) -> GND

Commit message: Layout started
Pushed for BOM
Parts:
- added C3: 10n, Capacitor_SMD:C_0603_1608Metric, F.Cu at (120.4, 89.1)
- added J4: Conn_01x03, Connector_Molex:Molex_PicoBlade_53261-0371_1x03-1MP_P1.25mm_Horizontal, F.Cu at (146.7, 80.0)
- added R15: 10k, Resistor_SMD:R_0402_1005Metric, F.Cu at (120.9, 79.4)
- C14, C18, C5, R10, R9, U4: moved to B.Cu
- C6: footprint Capacitor_SMD:C_0603_1608Metric -> Capacitor_SMD:C_0402_1005Metric
- D1, D2: value LED_Small -> LTST-C281KRKT; footprint LED_SMD:LED_0603_1608Metric -> LED_SMD:LED_0402_1005Metric; moved to B.Cu
- J1: footprint 53047-0410:530470410 -> Connector_Molex:Molex_PicoBlade_53047-0410_1x04_P1.25mm_Vertical
- J2: value USB_C_Receptacle_USB2.0_14P -> USB4105-GF-A-120; footprint Connector_USB:USB_C_Receptacle_GCT_USB4110 -> Connector_USB:USB_C_Receptacle_GCT_USB4105-xx-A_16P_TopMnt_Horizontal
- R11, R12: value 1.5k -> 1k; footprint Resistor_SMD:R_0603_1608Metric -> Resistor_SMD:R_0402_1005Metric; moved to B.Cu
- R6: footprint Resistor_SMD:R_0603_1608Metric -> Resistor_SMD:R_0402_1005Metric
- moved R7 85.4 mm to (142.5, 69.1), turned to -90 degrees
- moved C2 83.0 mm to (142.1, 86.7), turned to -45 degrees
- moved C9 80.6 mm to (140.9, 71.8), turned to -90 degrees
- moved C6 80.1 mm to (139.8, 64.2)
- moved R8 80.1 mm to (142.5, 71.2), turned to 90 degrees
- moved C14 79.1 mm to (143.3, 85.0), turned to 180 degrees
- moved R11 78.5 mm to (146.9, 83.7), turned to 90 degrees
- moved C5 77.7 mm to (138.2, 81.8), turned to -90 degrees
- moved R12 77.1 mm to (145.6, 85.0), turned to 90 degrees
- moved L2 76.2 mm to (143.1, 91.6), turned to 45 degrees
- moved R10 75.7 mm to (138.4, 79.0), turned to -90 degrees
- moved R9 75.2 mm to (138.4, 84.3), turned to 180 degrees
- moved C15 73.7 mm to (136.6, 94.5), turned to 90 degrees
- moved U3 72.4 mm to (139.7, 88.1), turned to 135 degrees
- moved R5 72.1 mm to (132.3, 88.7)
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Connections:
- net Net-(C18-Pad1) renamed /bat+
- C10 pad 1: Net-(U3-EN) -> GND
- C10 pad 2: GND -> +BATT
- D3 pad 2: unconnected-(D3-A-Pad2) -> GND
- D4 pad 2: unconnected-(D4-A-Pad2) -> GND
- J1 pad 1: /Bout2 -> /Bout1
- J1 pad 2: /Bout1 -> /Bout2
- U2 pad 17: /AIN1 -> /BIN2
- U2 pad 18: /AIN2 -> /BIN1
- U2 pad 19: /BIN1 -> /AIN2
- U2 pad 20: /BIN2 -> /AIN1
- U2 pad 23: unconnected-(U2-IO19-Pad23) -> /USB_D-
- U2 pad 24: /SCL -> /USB_D+
- U2 pad 25: /SDA -> unconnected-(U2-IO21-Pad25)
- U2 pad 37: unconnected-(U2-IO41-Pad37) -> /SCL
- U2 pad 38: unconnected-(U2-IO42-Pad38) -> /SDA
- U3 pad 6: Net-(U3-EN) -> +BATT
- U3 pad 7: Net-(U3-EN) -> GND
- U3 pad 8: Net-(U3-EN) -> +BATT
- U4 pad 1: Net-(U4-TS) -> /ts
Routing:
- net /USB_D-: track 0.00 -> 18.7 mm
- net /USB_D+: track 0.00 -> 18.1 mm
- net /BIN1: track 0.00 -> 16.3 mm
- net /BIN2: track 0.00 -> 14.6 mm
- net /AIN1: track 0.00 -> 11.0 mm
- net /Aout1: track 0.00 -> 9.94 mm
- net /AIN2: track 0.00 -> 9.71 mm
- net /Aout2: track 0.00 -> 8.57 mm
- net /Bout2: track 0.00 -> 7.48 mm
- net Net-(U6-AISEN): track 0.00 -> 7.03 mm
- net /SCL: track 0.00 -> 6.97 mm
- net /ts: track 0.00 -> 6.88 mm, vias 0 -> 1
- net /SDA: track 0.00 -> 6.86 mm
- net /Bout1: track 0.00 -> 6.12 mm
- net Net-(J2-SHIELD): track 0.00 -> 4.21 mm
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- added copper zone on F.Cu, net +3.3V
- added copper zone on F.Cu, net +BATT
- added copper zone on B.Cu, net /bat+
- added copper zone on F.Cu, net /bat+
- added copper zone on F.Cu, net Net-(U3-L1)
- added copper zone on F.Cu, net Net-(U3-L2)

Commit message: Finished layout
Parts:
- moved C16 6.64 mm to (126.3, 88.1)
- moved C15 5.06 mm to (134.8, 89.8)
- moved R12 2.58 mm to (147.4, 83.2), turned to 180 degrees
- moved R15 1.70 mm to (120.3, 77.8), turned to 180 degrees
- moved C19 1.70 mm to (137.2, 89.5), turned to -135 degrees
- moved R11 1.66 mm to (147.4, 82.1), turned to 180 degrees
- moved C17 0.61 mm to (138.1, 90.5), turned to -135 degrees
- moved C8 0.50 mm to (121.4, 65.0)
- moved D3 0.33 mm to (128.9, 89.8)
- moved D4 0.33 mm to (131.8, 89.8)
- moved R14 0.32 mm to (128.5, 88.4)
- moved R5 0.32 mm to (132.3, 88.4)
- moved C14 0.29 mm to (143.6, 84.9), turned to 0 degrees
- moved R3 0.22 mm to (113.7, 84.8)
- moved R4 0.22 mm to (113.7, 82.6)
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Connections:
- U2 pad 13: unconnected-(U2-IO9-Pad13) -> /nFAULT
- U2 pad 14: unconnected-(U2-IO10-Pad14) -> /nSLEEP
- U2 pad 21: /nSLEEP -> unconnected-(U2-IO17-Pad21)
- U2 pad 22: /nFAULT -> unconnected-(U2-IO18-Pad22)
Routing:
- net +3.3V: track 0.00 -> 62.6 mm, vias 0 -> 10
- net +BATT: track 2.42 -> 48.3 mm, vias 0 -> 17
- net VBUS: track 0.00 -> 26.4 mm, vias 0 -> 3
- net Net-(J2-SHIELD): track 4.21 -> 22.4 mm
- net /nFAULT: track 0.00 -> 11.6 mm, vias 0 -> 2
- net /nSLEEP: track 2.72 -> 6.99 mm
- net Net-(U6-BIN2): track 0.00 -> 3.96 mm, vias 0 -> 2
- net Net-(U2-EN): track 0.00 -> 3.74 mm
- net Net-(U4-ILIM): track 0.00 -> 2.68 mm
- net Net-(U4-ISET): track 0.00 -> 2.51 mm
- net GND: track 0.00 -> 1.82 mm, vias 6 -> 186
- net /ts: track 6.88 -> 6.03 mm
- net Net-(D1-A): track 2.02 -> 1.33 mm
- added copper zone on B.Cu, net +BATT
- added copper zone on B.Cu, net GND
- added copper zone on F.Cu, net GND

Commit message: FInal
Parts:
- added D5: ESD5Z5.0T1G, Diode_SMD:D_SOD-523, B.Cu at (131.8, 91.8)
Routing:
- net /nFAULT: track 11.6 -> 12.3 mm
- net GND: vias 186 -> 195
