File: Radiator valve/Radiator valve.kicad_sch (KiCad schematic)
At the start: 48 parts, among them J1 53047-0410, J2 USB4105-GF-A-120, J4 Conn_01x03, M1 Stepper_Motor, U1 MLX90632SLD-BCB-000-SP, U2 ESP32-S3-MINI-1, U3 TPS63031DSK, U4 BQ24075RGT, U6 DRV8833PW

Commit message: Finished layout
Connections:
- net nFAULT: now also U2.13 (IO9); no longer U2.22 (IO18)
- net nSLEEP: now also U2.14 (IO10); no longer U2.21 (IO17)
- no-connect marks 26 -> 30
Other:
- note removed: "m: link do mousera model: nazwa komponentu w mouserze"
Changed lines of the file:
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@@
+	)
+	(no_connect
+		(at 220.98 96.52)
 	)
 	(no_connect
@@
 	)
 	(no_connect
+		(at 254 73.66)
+	)
+	(no_connect
 		(at 220.98 71.12)
 	)
@@
 	)
 	(no_connect
+		(at 254 63.5)
+	)
+	(no_connect
 		(at 254 88.9)
 	)
@@
 	)
 	(no_connect
-		(at 220.98 76.2)
+		(at 254 66.04)
+	)
+	(no_connect
+		(at 220.98 93.98)
 	)
 	(no_connect
@@
 	)
 	(no_connect
-		(at 220.98 73.66)
+		(at 254 76.2)
 	)
 	(no_connect
@@
 	)
 	(rectangle
-		(start -63.754 138.938)
-		(end -12.7 179.07)
-		(stroke
-			(width 0)
-			(type default)
-		)
-		(fill
-			(type none)
-		)
-	)
-	(rectangle
 		(start 177.292 13.335)
 		(end 284.48 114.3)
@@
 	(rectangle
 		(start 219.456 114.3)
-		(end 238.76 146.304)
+		(end 243.332 146.304)
 		(stroke
 			(width 0)
@@
 		)
 	)
-	(text "m: link do mousera\nmodel: nazwa komponentu w mouserze\n"
-		(exclude_from_sim no)
-		(at -41.656 151.638 0)
-		(effects
-			(font
-				(size 1.27 1.27)
-			)
-		)
-	)
 	(text "stm\ncontrolling on off\nstate\n"
 		(exclude_from_sim no)
@@
 		)
 	)
+	(label "nFAULT"
+		(at 220.98 73.66 180)
+		(fields_autoplaced yes)
+		(effects
+			(font
+				(size 1.27 1.27)
+			)
+			(justify right bottom)
+		)
+	)
 	(label "bat+"
 		(at 142.24 151.13 0)
@@
 		)
 	)
+	(label "nSLEEP"
+		(at 220.98 76.2 180)
+		(fields_autoplaced yes)
+		(effects
+			(font
+				(size 1.27 1.27)
+			)
+			(justify right bottom)
+		)
+	)
 	(label "Aout2"
 		(at 138.43 62.23 0)
@@
 		)
 	)
-	(label "nSLEEP"
-		(at 220.98 93.98 180)
-		(fields_autoplaced yes)
-		(effects
-			(font
-				(size 1.27 1.27)
-			)
-			(justify right bottom)
-		)
-	)
 	(label "Bout1"
 		(at 152.4 67.31 180)
@@
 		)
 	)
-	(label "nFAULT"
-		(at 220.98 96.52 180)
-		(fields_autoplaced yes)
-		(effects
-			(font
-				(size 1.27 1.27)
-			)
-			(justify right bottom)
-		)
-	)

Commit message: FInal
Parts:
- added D5: ESD5Z5.0T1G, Diode_SMD:D_SOD-523, symbol Diode:ESD5Zxx
Connections:
- net GND: now also D5.2 (A)
- net VBUS: now also D5.1 (K)
Other:
- moved on the sheet: C12, C15, C16, D3, D4, J2, R14, R5
